File: hardware/pentabug_1layer.sch (EAGLE design)
At the start: 17 parts, among them IC1 ATMEGA88

Commit message: modified to use biggr buzzr - routing not adapted yet!
Parts:
- SG1: value MULTIBUZZR -> MULTIBUZZRTDKBUZZR; device buglbr:MULTIBUZZR -> buglbr:MULTIBUZZRTDKBUZZR
Changed lines of the file:
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@@
 <part name="JP2" library="pinhead" deviceset="PINHD-2X3" device=""/>
 <part name="U$1" library="buglbr" deviceset="VIBRAMOTOR" device=""/>
-<part name="SG1" library="buglbr" deviceset="MULTIBUZZR" device=""/>
+<part name="SG1" library="buglbr" deviceset="MULTIBUZZR" device="TDKBUZZR"/>
 <part name="GND10" library="supply1" deviceset="GND" device=""/>
 <part name="GND12" library="supply1" deviceset="GND" device=""/>
