File: hardware/pentabug_ir.brd (EAGLE design)
At the start: 86 x 33 mm, 26 parts, among them IC1 ATMEGA88

Commit message: some beautifications
Parts:
- JP3: device pinhead:1X05 -> pinhead:1X03
- JP5: device pinhead:1X03 -> pinhead:1X05
- moved JP3 27.3 mm to (29.2, 8.57)
- moved JP1 15.2 mm to (43.2, 2.54), turned to 180 degrees
- moved JP5 12.7 mm to (55.9, 2.54), turned to 0 degrees
- renumbered U$2 to IR
Connections:
- net PB1 renamed PB2
- removed net N$9: BAT1.+, JP5.3
- new net BAT: BAT1.+, JP1.3
- net +5V: now also JP1.1; no longer JP5.1
- net GND: now also JP3.3, JP5.5; no longer JP1.3, JP3.5
- net PD5: now also JP5.2; no longer JP3.2
- net PD6: now also JP5.3; no longer JP3.3
- net PD7: now also JP5.4; no longer JP3.4
- net RX: now also JP3.1; no longer JP1.1
- net TX: now also JP3.2; no longer JP1.2
- net VCC: now also JP1.2, JP5.1; no longer JP3.1, JP5.2
Routing:
- net GND: track 228.5 -> 201.9 mm, vias 2 -> 39
- net N$9: track 8.19 -> 0.00 mm
- net BAT: track 0.00 -> 8.19 mm
- net SCK: track 38.0 -> 41.2 mm
- net MISO: track 41.6 -> 43.5 mm
- net S2: track 32.8 -> 34.6 mm
- added copper zone on layer 1, net BAT
Other:
- board text added: "+5V"
- board text added: "BAT"
- board text added: "IR"
- board text added: "PB2"
- board text added: "PC4"
- board text added: "PC5"
- board text added: "SCL"
- board text added: "SDA"
- board text added: "bigalex@gmx.de"
- board text removed: "PD2"
- board text removed: "PD3"
- board text removed: "PD4"
- board text removed: "Pentabug V1.0"
