File: addons/ledmatrix.sch (EAGLE design)
At the start: 11 parts

Commit message: anpassen an neues board
Parts:
- LED1, LED2, LED3, LED4, LED5, LED6, LED7, LED8, LED9: device led:LED5MM -> SparkFun:LED5MM
Connections:
- net PD2 renamed PC5
- net PD3 renamed PC4
- net PD4 renamed PB2
