File: addons/pentatonic.sch (EAGLE design)
At the start: 12 parts

Commit message: anpassen an neues board
Parts:
- LED1, LED2, LED3, LED4, LED5: device led:LED5MM -> SparkFun:LED5MM
- S1, S2, S3, S4, S5: value (none) -> SWITCH-MOMENTARY-2PTH; device switch-omron:10-XX -> SparkFun:SWITCH-MOMENTARY-2PTH
Connections:
- removed net PD2: LED1.C, S1.S, S1.S1, SV1.2
- removed net PD3: LED2.C, S2.S, S2.S1, SV1.3
- removed net PD4: LED3.C, S3.S, S3.S1, SV1.4
- new net PB2: LED3.C, S3.2, SV1.4
- new net PC4: LED2.C, S2.2, SV1.3
- new net PC5: LED1.C, S1.2, SV1.2
- net GND: now also S1.1, S2.1, S3.1, S4.1, S5.1; no longer S1.P, S1.P1, S2.P, S2.P1, S3.P, S3.P1, S4.P, S4.P1, S5.P, S5.P1
- net PD5: now also S4.2; no longer S4.S, S4.S1
- net PD6: now also S5.2; no longer S5.S, S5.S1
