File: hardware/v2/pentabug_v2.brd (EAGLE design)
At the start: 166.7 x 33 mm, 49 parts, among them IC1 ATMEGA88

Commit message: fixes issue #6, correct values for r4 and r5
Parts:
- R4, R5: value 22R -> 33R
Changed lines of the file:
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@@
 <attribute name="VALUE" x="17.78" y="5.715" size="1.27" layer="27" ratio="10" rot="R270"/>
 </element>
-<element name="R4" library="rcl" package="0207/10" value="22R" x="10.16" y="6.55" smashed="yes" rot="R295">
+<element name="R4" library="rcl" package="0207/10" value="33R" x="10.16" y="6.55" smashed="yes" rot="R295">
 <attribute name="NAME" x="10.36350625" y="6.443071875" size="1.27" layer="25" font="vector" ratio="10" rot="SR115" align="center"/>
 <attribute name="VALUE" x="8.629121875" y="8.330434375" size="1.27" layer="27" ratio="10" rot="R295"/>
@@
 <attribute name="VALUE" x="4.709878125" y="11.562284375" size="1.27" layer="27" ratio="10" rot="R110"/>
 </element>
-<element name="R5" library="rcl" package="0207/10" value="22R" x="10.16" y="26.47" smashed="yes" rot="R65">
+<element name="R5" library="rcl" package="0207/10" value="33R" x="10.16" y="26.47" smashed="yes" rot="R65">
 <attribute name="NAME" x="10.34814375" y="25.30414375" size="1.27" layer="25" font="vector" ratio="10" rot="R65"/>
 <attribute name="VALUE" x="9.780134375" y="24.1528375" size="1.27" layer="27" ratio="10" rot="R65"/>

Commit message: correct labels in schematic for pentatonic fixes #7
Connections:
- net PB2_T renamed PD7_T
- net SCL renamed PC5/SCL
- net SDA renamed PC4/SDA
- net PC4_T: now also LED9.K, S7.1, S7.2, SV5.3; no longer LED6.K, S4.1, S4.2, SV4.3
- net PC5_T: now also LED8.K, S6.1, S6.2, SV5.2; no longer LED5.K, S3.1, S3.2, SV4.2
- net PD5_T: now also LED5.K, S3.1, S3.2, SV4.2; no longer LED8.K, S6.1, S6.2, SV5.2
- net PD6_T: now also LED6.K, S4.1, S4.2, SV4.3; no longer LED9.K, S7.1, S7.2, SV5.3
Routing:
- net PD6_T: track 35.3 -> 24.1 mm
- net PC4_T: track 24.1 -> 35.3 mm
Changed lines of the file:
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@@
 <?xml version="1.0" encoding="utf-8"?>
 <!DOCTYPE eagle SYSTEM "eagle.dtd">
-<eagle version="6.4">
+<eagle version="6.5.0">
 <drawing>
 <settings>
@@
 <layer number="19" name="Unrouted" color="6" fill="1" visible="yes" active="yes"/>
 <layer number="20" name="Dimension" color="15" fill="1" visible="no" active="yes"/>
-<layer number="21" name="tPlace" color="7" fill="1" visible="no" active="yes"/>
+<layer number="21" name="tPlace" color="7" fill="1" visible="yes" active="yes"/>
 <layer number="22" name="bPlace" color="7" fill="1" visible="no" active="yes"/>
 <layer number="23" name="tOrigins" color="15" fill="1" visible="no" active="yes"/>
 <layer number="24" name="bOrigins" color="15" fill="1" visible="no" active="yes"/>
-<layer number="25" name="tNames" color="7" fill="1" visible="no" active="yes"/>
+<layer number="25" name="tNames" color="7" fill="1" visible="yes" active="yes"/>
 <layer number="26" name="bNames" color="7" fill="1" visible="no" active="yes"/>
-<layer number="27" name="tValues" color="7" fill="1" visible="no" active="yes"/>
+<layer number="27" name="tValues" color="7" fill="1" visible="yes" active="yes"/>
 <layer number="28" name="bValues" color="7" fill="1" visible="no" active="yes"/>
 <layer number="29" name="tStop" color="7" fill="3" visible="no" active="yes"/>
@@
 <wire x1="57.15" y1="21.59" x2="57.15" y2="20.32" width="0.4064" layer="1"/>
 </signal>
-<signal name="SCL">
+<signal name="PC5/SCL">
 <contactref element="JP4" pad="2"/>
 <contactref element="IC1" pad="28"/>
@@
 <wire x1="27.94" y1="29.21" x2="28.575" y2="29.845" width="0.4064" layer="1"/>
 </signal>
-<signal name="SDA">
+<signal name="PC4/SDA">
 <contactref element="JP4" pad="3"/>
 <contactref element="IC1" pad="27"/>
@@
 </polygon>
 </signal>
-<signal name="PD5_T">
+<signal name="PC5_T">
 <contactref element="SV5" pad="2"/>
 <contactref element="LED8" pad="K"/>
@@
 <wire x1="116.84" y1="25.4" x2="118.745" y2="23.495" width="0.6096" layer="1"/>
 </signal>
-<signal name="PD6_T">
+<signal name="PC4_T">
 <contactref element="SV5" pad="3"/>
 <contactref element="LED9" pad="K"/>
@@
 <wire x1="110.49" y1="29.21" x2="110.49" y2="30.45" width="0.6096" layer="1"/>
 </signal>
-<signal name="PC5_T">
+<signal name="PD5_T">
 <contactref element="SV4" pad="2"/>
 <contactref element="LED5" pad="K"/>
@@
 <wire x1="98.7806" y1="9.1694" x2="98.7806" y2="10.7188" width="0.6096" layer="1"/>
 </signal>
-<signal name="PC4_T">
+<signal name="PD6_T">
 <contactref element="SV4" pad="3"/>
 <contactref element="LED6" pad="K"/>
@@
 <wire x1="110.49" y1="5.08" x2="110.49" y2="2.54" width="0.6096" layer="1"/>
 </signal>
-<signal name="PB2_T">
+<signal name="PD7_T">
 <contactref element="SV4" pad="4"/>
 <contactref element="LED7" pad="K"/>

Commit message: correct labels for ledmatrix nets fixes #8
Connections:
- net PB2_L: now also LED10.A, LED11.A, LED12.A, SV__5.4; no longer LED12.K, LED15.K, LED18.K, SV__4.4
- net PC4_L: now also LED13.A, LED14.A, LED15.A, SV__5.3; no longer LED11.K, LED14.K, LED17.K, SV__4.3
- net PC5_L: now also LED16.A, LED17.A, LED18.A, SV__5.2; no longer LED10.K, LED13.K, LED16.K, SV__4.2
- net PD5_L: now also LED10.K, LED13.K, LED16.K, SV__4.2; no longer LED16.A, LED17.A, LED18.A, SV__5.2
- net PD6_L: now also LED11.K, LED14.K, LED17.K, SV__4.3; no longer LED13.A, LED14.A, LED15.A, SV__5.3
- net PD7_L: now also LED12.K, LED15.K, LED18.K, SV__4.4; no longer LED10.A, LED11.A, LED12.A, SV__5.4
Routing:
- net PD5_L: track 30.8 -> 35.1 mm
- net PC5_L: track 35.1 -> 30.8 mm
- net PD7_L: track 25.1 -> 24.0 mm
- net PB2_L: track 24.0 -> 25.1 mm
Changed lines of the file:
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@@
 </polygon>
 </signal>
-<signal name="PC5_L">
+<signal name="PD5_L">
 <contactref element="SV__4" pad="2"/>
 <contactref element="LED10" pad="K"/>
@@
 <wire x1="144.5808" y1="15.70223125" x2="143.8142875" y2="14.935715625" width="0.6096" layer="1"/>
 </signal>
-<signal name="PC4_L">
+<signal name="PD6_L">
 <contactref element="SV__4" pad="3"/>
 <contactref element="LED11" pad="K"/>
@@
 <wire x1="144.78" y1="9.525" x2="144.78" y2="2.54" width="0.6096" layer="1"/>
 </signal>
-<signal name="PB2_L">
+<signal name="PD7_L">
 <contactref element="SV__4" pad="4"/>
 <contactref element="LED12" pad="K"/>
@@
 <wire x1="147.32" y1="5.08" x2="147.32" y2="2.54" width="0.6096" layer="1"/>
 </signal>
-<signal name="PD5_L">
+<signal name="PC5_L">
 <contactref element="SV__5" pad="2"/>
 <contactref element="LED18" pad="A"/>
@@
 <wire x1="152.663025" y1="9.896975" x2="152.663025" y2="7.62000625" width="0.6096" layer="16"/>
 </signal>
-<signal name="PD6_L">
+<signal name="PC4_L">
 <contactref element="SV__5" pad="3"/>
 <contactref element="LED15" pad="A"/>
@@
 <wire x1="157.602165625" y1="15.117834375" x2="157.602165625" y2="12.55914375" width="0.6096" layer="16"/>
 </signal>
-<signal name="PD7_L">
+<signal name="PB2_L">
 <contactref element="SV__5" pad="4"/>
 <contactref element="LED12" pad="A"/>
