File: hardware/v2/pentabug_v2.1.sch (EAGLE design)
At the start: 51 parts, among them IC1 ATMEGA88

Commit message: some improvent on placement of print and mounting holes for motor
Parts:
- removed R6: (no value), bigalexeasysolder:R-EU_EASY-SOLDER0207/10_EASY-SOLDER
- removed R7: 100K, bigalexeasysolder:R-EU_EASY-SOLDER0207/10_EASY-SOLDER
- IC1: value ATMEGA88 -> ATMEGA328P-PU
Other:
- note added: "Pentabug V2.1"
- note added: "voll kompatibel zu V2.0 Lötstellen+Beschriftung verbesert"
- note removed: "Pentabug V2.0"
Changed lines of the file:
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@@
 </classes>
 <parts>
-<part name="IC1" library="atmel" deviceset="MEGA8-P" device="" value="ATMEGA88"/>
+<part name="IC1" library="atmel" deviceset="MEGA8-P" device="" value="ATMEGA328P-PU"/>
 <part name="P+2" library="supply1" deviceset="VCC" device=""/>
 <part name="GND2" library="supply1" deviceset="GND" device=""/>
@@
 <part name="LED17" library="led" deviceset="LED" device="5MM"/>
 <part name="LED18" library="led" deviceset="LED" device="5MM"/>
-<part name="R6" library="bigalexeasysolder" deviceset="R-EU_EASY-SOLDER" device="0207/10_EASY-SOLDER"/>
-<part name="R7" library="bigalexeasysolder" deviceset="R-EU_EASY-SOLDER" device="0207/10_EASY-SOLDER" value="100K"/>
 </parts>
 <sheets>
@@
 <wire x1="157.48" y1="40.64" x2="205.74" y2="40.64" width="0.1524" layer="94"/>
 <text x="160.02" y="43.18" size="1.778" layer="94">Serielle Schnittstelle und ISP</text>
-<text x="127.508" y="-46.482" size="3.81" layer="94" font="vector">DEFEKT!</text>
+<text x="127.508" y="-50.8" size="3.81" layer="94" font="vector">DEFEKT!</text>
 <text x="104.14" y="43.18" size="1.778" layer="94">Vibrationsmotor und Treiber</text>
 <wire x1="157.48" y1="40.64" x2="101.6" y2="40.64" width="0.1524" layer="94"/>
@@
 <text x="104.14" y="-20.32" size="1.778" layer="94">Piezo Buzzer</text>
 <text x="160.02" y="-20.32" size="1.778" layer="94">Batterie und Spannungssensor</text>
-<text x="119.38" y="-38.1" size="3.81" layer="94">Pentabug V2.0</text>
+<text x="119.38" y="-38.1" size="3.81" layer="94">Pentabug V2.1</text>
+<text x="119.38" y="-41.91" size="1.27" layer="94">voll kompatibel zu V2.0
+Lötstellen+Beschriftung verbesert</text>
 </plain>
 <instances>
@@
 <instance part="P+8" gate="VCC" x="-22.86" y="106.68"/>
 <instance part="P+9" gate="VCC" x="55.88" y="2.54"/>
-<instance part="R6" gate="G$1" x="25.4" y="53.34"/>
-<instance part="R7" gate="G$1" x="-10.16" y="43.18"/>
 </instances>
 <busses>
@@
 </schematic>
 </drawing>
+<compatibility>
+<note version="6.3" minversion="6.2.2" severity="warning">
+Since Version 6.2.2 text objects can contain more than one line,
+which will not be processed correctly with this version.
+</note>
+</compatibility>
 </eagle>

Commit message: I can haz eazy solder transistors.
Parts:
- added SV1: (no value), con-lstb:MA05-2
- Q1, Q2: device transistors:2N7000_TO92 -> bigalexeasysolder:2N7000
Changed lines of the file:
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@@
 <part name="C3" library="resistor" deviceset="C-EU" device="025-024X044" value="100nF"/>
 <part name="GND11" library="supply1" deviceset="GND" device=""/>
-<part name="Q1" library="transistors" deviceset="2N700*" device="_TO92" technology="0"/>
+<part name="Q1" library="bigalexeasysolder" deviceset="2N700*" device="" technology="0"/>
 <part name="R3" library="bigalexeasysolder" deviceset="R-EU_EASY-SOLDER" device="0207/10_EASY-SOLDER" value="10k"/>
 <part name="LED1" library="SparkFun" deviceset="LED" device="5MM"/>
@@
 <part name="P+6" library="supply1" deviceset="VCC" device=""/>
 <part name="JP1" library="pinhead" deviceset="PINHD-1X3" device=""/>
-<part name="Q2" library="transistors" deviceset="2N700*" device="_TO92" technology="0"/>
+<part name="Q2" library="bigalexeasysolder" deviceset="2N700*" device="" technology="0"/>
 <part name="R4" library="bigalexeasysolder" deviceset="R-EU_EASY-SOLDER" device="0207/10_EASY-SOLDER" value="33R"/>
 <part name="IR" library="buglbr" deviceset="TSOP382" device=""/>
@@
 <part name="LED17" library="led" deviceset="LED" device="5MM"/>
 <part name="LED18" library="led" deviceset="LED" device="5MM"/>
+<part name="SV1" library="con-lstb" deviceset="MA05-2" device=""/>
 </parts>
 <sheets>
@@
 <instance part="P+8" gate="VCC" x="-22.86" y="106.68"/>
 <instance part="P+9" gate="VCC" x="55.88" y="2.54"/>
+<instance part="SV1" gate="G$1" x="55.88" y="40.64"/>
 </instances>
 <busses>

Commit message: v2.1 production files, updated docs, some cleanup
Parts:
- removed LED10, LED11, LED12, LED13, LED14, LED15, LED16, LED17, LED18, LED5, LED6, LED7, LED8, LED9: (no value), led:LED5MM
- removed S3, S4, S5, S6, S7: (no value), switch-omron:10-XX
- removed SV1: (no value), con-lstb:MA05-2
- removed SV4, SV5, SV__4, SV__5: (no value), con-lsta:FE05-1
Connections:
- removed net GND_L: SV__4.5, SV__5.5
- removed net GND_M: S3.P, S3.P1, S4.P, S4.P1, S5.P, S5.P1, S6.P, S6.P1, S7.P, S7.P1, SV4.5, SV5.5
- removed net PB2_L: LED10.A, LED11.A, LED12.A, SV__5.4
- removed net PC4_L: LED13.A, LED14.A, LED15.A, SV__5.3
- removed net PC4_T: LED9.C, S7.S, S7.S1, SV5.3
- removed net PC5_L: LED16.A, LED17.A, LED18.A, SV__5.2
- removed net PC5_T: LED8.C, S6.S, S6.S1, SV5.2
- removed net PD5_L: LED10.C, LED13.C, LED16.C, SV__4.2
- removed net PD5_T: LED5.C, S3.S, S3.S1, SV4.2
- removed net PD6_L: LED11.C, LED14.C, LED17.C, SV__4.3
- removed net PD6_T: LED6.C, S4.S, S4.S1, SV4.3
- removed net PD7_L: LED12.C, LED15.C, LED18.C, SV__4.4
- removed net PD7_T: LED7.C, S5.S, S5.S1, SV4.4
- removed net VCC_L: SV__4.1, SV__5.1
- removed net VCC_M: LED5.A, LED6.A, LED7.A, LED8.A, LED9.A, SV5.1
